Commit message: Updated 4dof manipulator with end-effector joint, and with new inertias. Updated plotting function.

File: URDF_models/floating_planar_4dof_manipulator.urdf (robot description, URDF)
Before this commit: robot floating_planar_4dof_manipulator, 5 links, 4 joints
Links:
- added link EndEffector, mass 0.1; collision sphere radius=0.05; visual sphere radius=0.05
- link Chaser_Base: mass 50.0 -> 150.0
- link Link_1: mass 3.0 -> 5.0
- link Link_2: mass 3.0 -> 5.0
- link Link_3: mass 3.0 -> 5.0
- link Link_4: mass 3.0 -> 5.0
Joints:
- added joint Joint_5_EE: type fixed, parent Link_4, child EndEffector, origin xyz=0.5 0 0 rpy=0 0 0

Commit message: Updated EE mass to 1 kg.

File: URDF_models/floating_planar_4dof_manipulator.urdf (robot description, URDF)
Before this commit: robot floating_planar_4dof_manipulator, 6 links, 5 joints
Links:
- link Chaser_Base: mass 150.0 -> 300.0
- link EndEffector: mass 0.1 -> 1.0

Commit message: Updated spherical collisions

File: URDF_models/floating_planar_4dof_manipulator.urdf (robot description, URDF)
Before this commit: robot floating_planar_4dof_manipulator, 6 links, 5 joints
Links:
- link Chaser_Base: geometry visual box size=0.5 0.5 0
- link EndEffector: geometry collision sphere radius=0.03; visual sphere radius=0.05
- link Link_1: geometry collision sphere radius=0.03; collision sphere radius=0.03
- link Link_2: geometry collision sphere radius=0.03; collision sphere radius=0.03
- link Link_3: geometry collision sphere radius=0.03; collision sphere radius=0.03
- link Link_4: geometry collision sphere radius=0.03; collision sphere radius=0.03
