Commit message: Update revolute to continuous joint

File: URDF_models/ChaserRobot.urdf (robot description, URDF)
Before this commit: robot Chaser_Robot, 9 links, 8 joints
Joints:
- joint Joint_1: type revolute -> continuous
- joint Joint_2: type revolute -> continuous
- joint Joint_3: type revolute -> continuous
- joint Joint_4: type revolute -> continuous
- joint Joint_5: type revolute -> continuous
- joint Joint_6: type revolute -> continuous
- joint Joint_7: type revolute -> continuous
