Commit message: Added joint limits

File: SPARTpy/urdf/floating_7dof_manipulator.urdf (robot description, URDF)
Before this commit: robot Chaser_Robot, 9 links, 8 joints
Joints:
- joint Joint_1: limit (none) -> lower=-1e9 upper=1e9 effort=1e9 velocity=1e9
- joint Joint_2: limit (none) -> lower=-1e9 upper=1e9 effort=1e9 velocity=1e9
- joint Joint_3: limit (none) -> lower=-1e9 upper=1e9 effort=1e9 velocity=1e9
- joint Joint_4: limit (none) -> lower=-1e9 upper=1e9 effort=1e9 velocity=1e9
- joint Joint_5: limit (none) -> lower=-1e9 upper=1e9 effort=1e9 velocity=1e9
- joint Joint_6: limit (none) -> lower=-1e9 upper=1e9 effort=1e9 velocity=1e9
- joint Joint_7: limit (none) -> lower=-1e9 upper=1e9 effort=1e9 velocity=1e9

File: URDF_models/floating_7dof_manipulator.urdf (robot description, URDF)
Before this commit: robot Chaser_Robot, 9 links, 8 joints
Joints:
- joint Joint_1: limit (none) -> effort=1e9 velocity=1e9
- joint Joint_2: limit (none) -> effort=1e9 velocity=1e9
- joint Joint_3: limit (none) -> effort=1e9 velocity=1e9
- joint Joint_4: limit (none) -> effort=1e9 velocity=1e9
- joint Joint_5: limit (none) -> effort=1e9 velocity=1e9
- joint Joint_6: limit (none) -> effort=1e9 velocity=1e9
- joint Joint_7: limit (none) -> effort=1e9 velocity=1e9
- joint Joint_EE: limit (none) -> effort=1e9 velocity=1e9

Commit message: Added limits on second joints to avoid singularities.

File: SPARTpy/urdf/floating_7dof_manipulator.urdf (robot description, URDF)
Before this commit: robot Chaser_Robot, 9 links, 8 joints
Joints:
- joint Joint_2: limit lower=-1e9 upper=1e9 effort=1e9 velocity=1e9 -> lower=-3.14159 upper=-0.17453 effort=1e9 velocity=1e9

File: URDF_models/floating_7dof_manipulator.urdf (robot description, URDF)
Before this commit: robot Chaser_Robot, 9 links, 8 joints
Joints:
- joint Joint_2: limit effort=1e9 velocity=1e9 -> lower=-3.14159 upper=-0.17453 effort=1e9 velocity=1e9; type continuous -> revolute

Commit message: Removed joint limits in urdf, enforced via SCP

File: SPARTpy/urdf/floating_7dof_manipulator.urdf (robot description, URDF)
Before this commit: robot Chaser_Robot, 9 links, 8 joints
Joints:
- joint Joint_2: limit lower=-3.14159 upper=-0.17453 effort=1e9 velocity=1e9 -> effort=1e9 velocity=1e9; type revolute -> continuous

File: URDF_models/floating_7dof_manipulator.urdf (robot description, URDF)
Before this commit: robot Chaser_Robot, 9 links, 8 joints
Joints:
- joint Joint_2: limit lower=-3.14159 upper=-0.17453 effort=1e9 velocity=1e9 -> effort=1e9 velocity=1e9; type revolute -> continuous
